File: Motor Control - Inverter.kicad_sch (KiCad schematic)
At the start: 54 parts, among them J3 Phase A, J4 Phase B, J5 Phase C, Q1 TPW1R306PL,L1Q, Q2 TPW1R306PL,L1Q, Q3 TPW1R306PL,L1Q, Q4 TPW1R306PL,L1Q, Q5 TPW1R306PL,L1Q, Q6 TPW1R306PL,L1Q

Commit message: Kicad 10
Parts:
- renumbered C8 to C133, C8 to C134, C8 to C135, C8 to C136, C8 to C137, C8 to C138, D17 to D10, D17 to D11, D17 to D3, D17 to D4, D17 to D5, D17 to D6, D17 to D7, D17 to D8, D17 to D9, R23 to R55, R23 to R56, R23 to R57, R23 to R58, R23 to R59, R23 to R60
