File: Power - Generation.kicad_sch (KiCad schematic)
At the start: 110 parts, among them U2 LMR36506MSC5RPERQ1, U3 LMR36006FSCQ, U4 TPS62172DSG, U5 LP2992IM5-3.3/NOPB

Commit message: Kicad 10
Parts:
- renumbered R28 to R7
